File: hardware/microcontroller.kicad_sch (KiCad schematic)
At the start: 12 parts, among them J1 AVR-ISP-6, SW2 SKRPACE010, U1 ATmega328P-A, Y2 Crystal-32kHz

Commit message: Removed comments on UART, added some footprints and started fixing rule checks
Parts:
- C5: Manuf. Part # (none) -> GRM21BR71H104KA01L; Part Num GRM21BR71H104KA01L -> (none); Price/unit $0.0097 -> (none); Supplier Name (none) -> JLCPCB; Supplier Unit Price (none) -> $0.0097
- R3: Manuf. Part # (none) -> 0805W8F1002T5E; Part Num 0805W8F1002T5E -> (none); Price/unit $0.0017 -> (none); Supplier Name (none) -> JLCPCB; Supplier Unit Price (none) -> $0.0017
- SW2: Manuf. Name (none) -> ALPS Electric; Manuf. Part # (none) -> SKRPACE010; Manufacturer_Name ALPS Electric -> (none); Manufacturer_Part_Number SKRPACE010 -> (none); Mouser Part Number 688-SKRPACE010 -> (none); Mouser Price/Stock https://www.mouser.co.uk/ProductDetail/Alps-Alpine/SKRPACE0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 -> (none); Part Num SKRPACE010 -> (none); Price/unit $0.0573 -> (none); Supplier Name (none) -> JLCPCB; Supplier Unit Price (none) -> $0.0573
- U1: Manuf. Part # (none) -> ATMEGA328P-AU; Part Num ATMEGA328P-AU -> (none); Price/unit $2.2845 -> (none); Supplier Name (none) -> JLCPCB; Supplier Unit Price (none) -> $2.2845
- Y2: Manuf. Name (none) -> HCI; Manuf. Part # (none) -> FL26T2-32.000-NTLLLDTL; Manufacturer_Name HCI -> (none); Manufacturer_Part_Number FL26T2-32.000-NTLLLDTL -> (none); Part Num FL26T2-32.000-NTLLLDTL -> (none); Price/unit $0.2669 -> (none); Supplier Name (none) -> JLCPCB; Supplier Unit Price (none) -> $0.2669
Changed lines of the file:
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@@
-			)
-		)
-		(property "Manufacturer_Name" "HCI"
-			(at 738.76 67.31 0)
-			(effects
-				(font
-					(size 1.27 1.27)
-				)
-				(justify left top)
-				(hide yes)
-			)
-		)
-		(property "Manufacturer_Part_Number" " FL26T2-32.000-NTLLLDTL"
-			(at 838.76 67.31 0)
-			(effects
-				(font
-					(size 1.27 1.27)
-				)
-				(justify left top)
-				(hide yes)
-			)
-		)
-		(property "Mouser Part Number" ""
-			(at 938.76 67.31 0)
-			(effects
-				(font
-					(size 1.27 1.27)
-				)
-				(justify left top)
-				(hide yes)
-			)
-		)
-		(property "Mouser Price/Stock" ""
-			(at 1038.76 67.31 0)
-			(effects
-				(font
-					(size 1.27 1.27)
-				)
-				(justify left top)
-				(hide yes)
 			)
 		)
@@
 			)
 		)
-		(property "Price/unit" " $0.2669"
+		(property "Package" " DT-26"
 			(at 242.57 76.2 0)
 			(effects
@@
 			)
 		)
-		(property "Part Num" " FL26T2-32.000-NTLLLDTL"
+		(property "Manuf. Name" "HCI"
 			(at 242.57 76.2 0)
 			(effects
@@
 			)
 		)
-		(property "Package" " DT-26"
+		(property "Manuf. Part #" " FL26T2-32.000-NTLLLDTL"
+			(at 242.57 76.2 0)
+			(effects
+				(font
+					(size 1.27 1.27)
+				)
+				(hide yes)
+			)
+		)
+		(property "Supplier Name" "JLCPCB"
+			(at 242.57 76.2 0)
+			(effects
+				(font
+					(size 1.27 1.27)
+				)
+				(hide yes)
+			)
+		)
+		(property "Supplier Unit Price" " $0.2669"
 			(at 242.57 76.2 0)
 			(effects
@@
 			)
 		)
+		(property "Supplier Name" ""
+			(at 36.83 74.93 0)
+			(effects
+				(font
+					(size 1.27 1.27)
+				)
+				(hide yes)
+			)
+		)
 		(pin "3"
 		)
@@
 			)
 		)
-		(property "Price/unit" "$0.0017"
+		(property "Package" "0805"
 			(at 46.99 118.11 0)
 			(effects
@@
 			)
 		)
-		(property "Part Num" "0805W8F1002T5E"
+		(property "Supplier Name" "JLCPCB"
 			(at 46.99 118.11 0)
 			(effects
@@
 			)
 		)
-		(property "Package" "0805"
+		(property "Manuf. Part #" "0805W8F1002T5E"
+			(at 46.99 118.11 0)
+			(effects
+				(font
+					(size 1.27 1.27)
+				)
+				(hide yes)
+			)
+		)
+		(property "Supplier Unit Price" "$0.0017"
 			(at 46.99 118.11 0)
 			(effects
@@
 			)
 		)
+		(property "Supplier Name" ""
+			(at 241.3 34.29 0)
+			(effects
+				(font
+					(size 1.27 1.27)
+				)
+				(hide yes)
+			)
+		)
 		(pin "2"
 		)
@@
 			)
 		)
+		(property "Supplier Name" ""
+			(at 250.19 76.2 0)
+			(effects
+				(font
+					(size 1.27 1.27)
+				)
+				(hide yes)
+			)
+		)
 		(pin "1"
 		)
@@
 			)
 		)
-		(property "Part Num" "GRM21BR71H104KA01L"
+		(property "Supplier Link" "https://jlcpcb.com/partdetail/MurataElectronics-GRM21BR71H104KA01L/C77082"
 			(at 40.64 125.73 0)
 			(effects
@@
 			)
 		)
-		(property "Price/unit" "$0.0097"
+		(property "Supplier Name" "JLCPCB"
 			(at 40.64 125.73 0)
 			(effects
@@
 			)
 		)
-		(property "Supplier Link" "https://jlcpcb.com/partdetail/MurataElectronics-GRM21BR71H104KA01L/C77082"
+		(property "Manuf. Part #" "GRM21BR71H104KA01L"
+			(at 40.64 125.73 0)
+			(effects
+				(font
+					(size 1.27 1.27)
+				)
+				(hide yes)
+			)
+		)
+		(property "Supplier Unit Price" "$0.0097"
 			(at 40.64 125.73 0)
 			(effects
@@
 			)
 		)
-		(property "Price/unit" "$2.2845"
-			(at 168.91 99.06 0)
-			(effects
-				(font
-					(size 1.27 1.27)
-				)
-				(hide yes)
-			)
-		)
-		(property "Part Num" "ATMEGA328P-AU"
-			(at 168.91 99.06 0)
-			(effects
-				(font
-					(size 1.27 1.27)
-				)
-				(hide yes)
-			)
-		)
 		(property "Package" "TQFP-32(7x7)"
 			(at 168.91 99.06 0)
+			(effects
+				(font
+					(size 1.27 1.27)
+				)
+				(hide yes)
+			)
+		)
+		(property "Supplier Name" "JLCPCB"
+			(at 168.91 99.06 0)
+			(effects
+				(font
+					(size 1.27 1.27)
+				)
+				(hide yes)
+			)
+		)
+		(property "Manuf. Part #" "ATMEGA328P-AU"
+			(at 168.148 103.124 0)
+			(effects
+				(font
+					(size 1.27 1.27)
+				)
+				(hide yes)
+			)
+		)
+		(property "Supplier Unit Price" "$2.2845"
+			(at 168.402 92.964 0)
 			(effects
 				(font
@@
 			)
 		)
-		(property "Sim.Device" "D"
+		(property "Sim.Pins" "1=K 2=A"
 			(at 50.8 118.11 0)
 			(effects
@@
 			)
 		)
-		(property "Sim.Pins" "1=K 2=A"
+		(property "Supplier Name" ""
 			(at 50.8 118.11 0)
 			(effects
@@
 			)
 		)
+		(property "Supplier Name" ""
+			(at 250.19 66.04 0)
+			(effects
+				(font
+					(size 1.27 1.27)
+				)
+				(hide yes)
+			)
+		)
 		(pin "1"
 		)
@@
 		)
 		(property "Description" "Resistor, small symbol"
+			(at 34.29 130.81 0)
+			(effects
+				(font
+					(size 1.27 1.27)
+				)
+				(hide yes)
+			)
+		)
+		(property "Supplier Name" ""
 			(at 34.29 130.81 0)
 			(effects
@@
 			)
 		)
-		(property "Mouser Part Number" "688-SKRPACE010"
-			(at 104.14 563.5 0)
-			(effects
-				(font
-					(size 1.27 1.27)
-				)
-				(justify left top)
-				(hide yes)
-			)
-		)
-		(property "Mouser Price/Stock" "https://www.mouser.co.uk/ProductDetail/Alps-Alpine/SKRPACE010?qs=dHDuPHwQO79W8iY66hDbLQ%3D%3D"
-			(at 104.14 663.5 0)
-			(effects
-				(font
-					(size 1.27 1.27)
-				)
-				(justify left top)
-				(hide yes)
-			)
-		)
-		(property "Manufacturer_Name" "ALPS Electric"
-			(at 104.14 763.5 0)
-			(effects
-				(font
-					(size 1.27 1.27)
-				)
-				(justify left top)
-				(hide yes)
-			)
-		)
-		(property "Manufacturer_Part_Number" "SKRPACE010"
-			(at 104.14 863.5 0)
-			(effects
-				(font
-					(size 1.27 1.27)
-				)
-				(justify left top)
-				(hide yes)
-			)
-		)
 		(property "Supplier Link" "https://jlcpcb.com/partdetail/Alpsalpine-SKRPACE010/C139797"
 			(at 120.65 68.58 0)
@@
 			)
 		)
-		(property "Price/unit" " $0.0573"
+		(property "Package" "SMD"
 			(at 120.65 68.58 0)
 			(effects
@@
 			)
 		)
-		(property "Part Num" "SKRPACE010"
+		(property "Manuf. Name" "ALPS Electric"
 			(at 120.65 68.58 0)
 			(effects
@@
 			)
 		)
-		(property "Package" "SMD"
+		(property "Manuf. Part #" "SKRPACE010"
+			(at 120.65 68.58 0)
+			(effects
+				(font
+					(size 1.27 1.27)
+				)
+				(hide yes)
+			)
+		)
+		(property "Supplier Name" "JLCPCB"
+			(at 120.65 68.58 0)
+			(effects
+				(font
+					(size 1.27 1.27)
+				)
+				(hide yes)
+			)
+		)
+		(property "Supplier Unit Price" " $0.0573"
 			(at 120.65 68.58 0)
 			(effects
@@
 			(at 254 34.29 0)
 			(effects
+				(font
+					(size 1.27 1.27)
+				)
+				(hide yes)
+			)
+		)
+		(property "Supplier Name" ""
+			(at 254 34.29 0)
+			(effects
